Commit message: Edited macro xacro, Modified launches files, joint yaml

File: servorobot_support/urdf/servorobotarm_macro.xacro (robot description, xacro)
@@ -13,5 +13,6 @@
         <visual>
             <geometry>
-                <mesh filename="package://servorobot_support/meshes/servorobot_arm/visual/servorobotarm_base.stl"/>
+                <mesh filename="package://servorobot_support/meshes/servorobot_arm/visual/servorobotarm_base.stl"
+                  scale="0.01 0.01 0.01"/>
             </geometry>
             <material name="servo_slategrey"/>
@@ -19,5 +20,6 @@
         <collision>
             <geometry>
-                <mesh filename="package://servorobot_support/meshes/servorobot_arm/collision/servorobotarm_base.stl"/>
+                <mesh filename="package://servorobot_support/meshes/servorobot_arm/collision/servorobotarm_base.stl"
+                  scale="0.01 0.01 0.01"/>
             </geometry>
         </collision>
@@ -26,5 +28,6 @@
         <visual>
             <geometry>
-                <mesh filename="package://servorobot_support/meshes/servorobot_arm/visual/servorobotarm_link_1.stl"/>
+                <mesh filename="package://servorobot_support/meshes/servorobot_arm/visual/servorobotarm_link_1.stl"
+                  scale="0.01 0.01 0.01"/>
             </geometry>
             <material name="servo_slategrey"/>
@@ -32,5 +35,6 @@
         <collision>
             <geometry>
-                <mesh filename="package://servorobot_support/meshes/servorobot_arm/collision/servorobotarm_link_1.stl"/>
+                <mesh filename="package://servorobot_support/meshes/servorobot_arm/collision/servorobotarm_link_1.stl"
+                  scale="0.01 0.01 0.01"/>
             </geometry>
         </collision>
@@ -39,5 +43,6 @@
         <visual>
             <geometry>
-                <mesh filename="package://servorobot_support/meshes/servorobot_arm/visual/servorobotarm_link_2.stl"/>
+                <mesh filename="package://servorobot_support/meshes/servorobot_arm/visual/servorobotarm_link_2.stl"
+                  scale="0.01 0.01 0.01"/>
             </geometry>
             <material name="servo_slategrey"/>
@@ -45,5 +50,6 @@
         <collision>
             <geometry>
-                <mesh filename="package://servorobot_support/meshes/servorobot_arm/collision/servorobotarm_link_2.stl"/>
+                <mesh filename="package://servorobot_support/meshes/servorobot_arm/collision/servorobotarm_link_2.stl"
+                  scale="0.01 0.01 0.01"/>
             </geometry>
         </collision>
@@ -52,5 +58,6 @@
         <visual>
             <geometry>
-                <mesh filename="package://servorobot_support/meshes/servorobot_arm/visual/servorobotarm_link_3.stl"/>
+                <mesh filename="package://servorobot_support/meshes/servorobot_arm/visual/servorobotarm_link_3.stl"
+                  scale="0.01 0.01 0.01"/>
             </geometry>
             <material name="servo_slategrey"/>
@@ -58,5 +65,6 @@
         <collision>
             <geometry>
-                <mesh filename="package://servorobot_support/meshes/servorobot_arm/collision/servorobotarm_link_3.stl"/>
+                <mesh filename="package://servorobot_support/meshes/servorobot_arm/collision/servorobotarm_link_3.stl"
+                  scale="0.01 0.01 0.01"/>
             </geometry>
         </collision>
@@ -65,5 +73,6 @@
         <visual>
             <geometry>
-                <mesh filename="package://servorobot_support/meshes/servorobot_arm/visual/servorobotarm_link_4.stl"/>
+                <mesh filename="package://servorobot_support/meshes/servorobot_arm/visual/servorobotarm_link_4.stl"
+                  scale="0.01 0.01 0.01"/>
             </geometry>
             <material name="servo_slategrey"/>
@@ -71,5 +80,6 @@
         <collision>
             <geometry>
-                <mesh filename="package://servorobot_support/meshes/servorobot_arm/collision/servorobotarm_link_4.stl"/>
+                <mesh filename="package://servorobot_support/meshes/servorobot_arm/collision/servorobotarm_link_4.stl"
+                  scale="0.01 0.01 0.01"/>
             </geometry>
         </collision>
@@ -78,5 +88,6 @@
         <visual>
             <geometry>
-                <mesh filename="package://servorobot_support/meshes/servorobot_arm/visual/servorobotarm_link_5.stl"/>
+                <mesh filename="package://servorobot_support/meshes/servorobot_arm/visual/servorobotarm_link_5.stl"
+                  scale="0.01 0.01 0.01"/>
             </geometry>
             <material name="servo_slategrey"/>
@@ -84,5 +95,6 @@
         <collision>
             <geometry>
-                <mesh filename="package://servorobot_support/meshes/servorobot_arm/collision/servorobotarm_link_5.stl"/>
+                <mesh filename="package://servorobot_support/meshes/servorobot_arm/collision/servorobotarm_link_5.stl"
+                  scale="0.01 0.01 0.01"/>
             </geometry>
         </collision>
@@ -91,5 +103,6 @@
         <visual>
             <geometry>
-                <mesh filename="package://servorobot_support/meshes/servorobot_arm/visual/servorobotarm_link_6.stl"/>
+                <mesh filename="package://servorobot_support/meshes/servorobot_arm/visual/servorobotarm_link_6.stl"
+                  scale="0.01 0.01 0.01"/>
             </geometry>
             <material name="servo_slategrey"/>
@@ -97,5 +110,6 @@
         <collision>
             <geometry>
-                <mesh filename="package://servorobot_support/meshes/servorobot_arm/collision/servorobotarm_link_6.stl"/>
+                <mesh filename="package://servorobot_support/meshes/servorobot_arm/collision/servorobotarm_link_6.stl"
+                  scale="0.01 0.01 0.01"/>
             </geometry>
         </collision>
@@ -106,5 +120,5 @@
         <parent link="${prefix}base_link"/>
         <child link="${prefix}link_1"/>
-        <origin xyz="0 0 0.450" rpy="0 0 0"/>
+        <origin xyz="0.105 0 0.955" rpy="0 0 0"/>
         <axis xyz="0 0 1"/>
         <limit lower="-3.1415" upper="3.1415" effort="0" velocity="2.9671"/>
@@ -113,5 +127,5 @@
       <parent link="${prefix}link_1"/>
       <child link="${prefix}link_2"/>
-      <origin xyz="0.320 0 0" rpy="0 0 0"/>
+      <origin xyz="-0.1 0 0.13" rpy="0 0 0"/>
       <axis xyz="0 1 0"/>
       <limit lower="-1.5707" upper="2.7052" effort="0" velocity="2.4434"/>
@@ -120,5 +134,5 @@
       <parent link="${prefix}link_2"/>
       <child link="${prefix}link_3"/>
-      <origin xyz="0 0 0.870" rpy="0 0 0"/>
+      <origin xyz="0 0 1" rpy="0 0 0"/>
       <axis xyz="0 -1 0"/>
       <limit lower="-3.1415" upper="3.1415" effort="0" velocity="2.7925"/>
@@ -127,5 +141,5 @@
       <parent link="${prefix}link_3"/>
       <child link="${prefix}link_4"/>
-      <origin xyz="0 0 0.225" rpy="0 0 0"/>
+      <origin xyz="0.46 0 0.26" rpy="0 0 0"/>
       <axis xyz="-1 0 0"/>
       <limit lower="-6.2831" upper="6.2831" effort="0" velocity="4.0142"/>
@@ -134,5 +148,5 @@
       <parent link="${prefix}link_4"/>
       <child link="${prefix}link_5"/>
-      <origin xyz="1.015 0 0" rpy="0 0 0"/>
+      <origin xyz="0.5 0 0" rpy="0 0 0"/>
       <axis xyz="0 -1 0"/>
       <limit lower="-2.1816" upper="2.1816" effort="0" velocity="4.0142"/>
@@ -141,5 +155,5 @@
       <parent link="${prefix}link_5"/>
       <child link="${prefix}link_6"/>
-      <origin xyz="0.175 0 0" rpy="0 0 0"/>
+      <origin xyz="0.7 0 0.01" rpy="0 0 0"/>
       <axis xyz="-1 0 0"/>
       <limit lower="-6.2831" upper="6.2831" effort="0" velocity="6.1086"/>
@@ -149,8 +163,15 @@
     <link name="${prefix}base" />
     <joint name="${prefix}base_link-base" type="fixed">
-        <origin xyz="0 0 0.450" rpy="0 0 0"/>
+        <origin xyz="0.105 0 0.955" rpy="0 0 0"/>
         <parent link="${prefix}base_link"/>
         <child link="${prefix}base"/>
     </joint>
+    <!-- ROS-Industrial 'tool0' frame: all-zeros tool frame -->
+    <link name="${prefix}tool0" />
+    <joint name="${prefix}link_6-tool0" type="fixed">
+      <origin xyz="0 0 0" rpy="${pi} ${-pi/2.0} 0" />
+      <parent link="${prefix}link_6" />
+      <child link="${prefix}tool0" />
+    </joint>
   </xacro:macro>
 </robot>

Commit message: Revised link_1 and joint_1

File: servorobot_support/urdf/servorobotarm_macro.xacro (robot description, xacro)
@@ -120,5 +120,5 @@
         <parent link="${prefix}base_link"/>
         <child link="${prefix}link_1"/>
-        <origin xyz="0.105 0 0.955" rpy="0 0 0"/>
+        <origin xyz="0.0 0 0.96" rpy="0 0 0"/>
         <axis xyz="0 0 1"/>
         <limit lower="-3.1415" upper="3.1415" effort="0" velocity="2.9671"/>
@@ -127,5 +127,5 @@
       <parent link="${prefix}link_1"/>
       <child link="${prefix}link_2"/>
-      <origin xyz="-0.1 0 0.13" rpy="0 0 0"/>
+      <origin xyz="0 0 0.13" rpy="0 0 0"/>
       <axis xyz="0 1 0"/>
       <limit lower="-1.5707" upper="2.7052" effort="0" velocity="2.4434"/>
@@ -163,5 +163,5 @@
     <link name="${prefix}base" />
     <joint name="${prefix}base_link-base" type="fixed">
-        <origin xyz="0.105 0 0.955" rpy="0 0 0"/>
+        <origin xyz="0.0 0 0.96" rpy="0 0 0"/>
         <parent link="${prefix}base_link"/>
         <child link="${prefix}base"/>

Commit message: Edited joint axis normal

File: servorobot_support/urdf/servorobotarm_macro.xacro (robot description, xacro)
@@ -128,5 +128,5 @@
       <child link="${prefix}link_2"/>
       <origin xyz="0 0 0.13" rpy="0 0 0"/>
-      <axis xyz="0 1 0"/>
+      <axis xyz="0 -1 0"/>
       <limit lower="-1.5707" upper="2.7052" effort="0" velocity="2.4434"/>
     </joint>
@@ -135,5 +135,5 @@
       <child link="${prefix}link_3"/>
       <origin xyz="0 0 1" rpy="0 0 0"/>
-      <axis xyz="0 -1 0"/>
+      <axis xyz="0 1 0"/>
       <limit lower="-3.1415" upper="3.1415" effort="0" velocity="2.7925"/>
     </joint>
@@ -142,5 +142,5 @@
       <child link="${prefix}link_4"/>
       <origin xyz="0.46 0 0.26" rpy="0 0 0"/>
-      <axis xyz="-1 0 0"/>
+      <axis xyz="1 0 0"/>
       <limit lower="-6.2831" upper="6.2831" effort="0" velocity="4.0142"/>
     </joint>
@@ -149,5 +149,5 @@
       <child link="${prefix}link_5"/>
       <origin xyz="0.5 0 0" rpy="0 0 0"/>
-      <axis xyz="0 -1 0"/>
+      <axis xyz="0 1 0"/>
       <limit lower="-2.1816" upper="2.1816" effort="0" velocity="4.0142"/>
     </joint>
@@ -156,5 +156,5 @@
       <child link="${prefix}link_6"/>
       <origin xyz="0.7 0 0.01" rpy="0 0 0"/>
-      <axis xyz="-1 0 0"/>
+      <axis xyz="1 0 0"/>
       <limit lower="-6.2831" upper="6.2831" effort="0" velocity="6.1086"/>
     </joint>

Commit message: Corrected joint limits

File: servorobot_support/urdf/servorobotarm_macro.xacro (robot description, xacro)
@@ -129,5 +129,5 @@
       <origin xyz="0 0 0.13" rpy="0 0 0"/>
       <axis xyz="0 -1 0"/>
-      <limit lower="-1.5707" upper="2.7052" effort="0" velocity="2.4434"/>
+      <limit lower="-1.5707" upper="1.5707" effort="0" velocity="2.4434"/>
     </joint>
     <joint name="${prefix}joint_3" type="revolute">
@@ -136,5 +136,5 @@
       <origin xyz="0 0 1" rpy="0 0 0"/>
       <axis xyz="0 1 0"/>
-      <limit lower="-3.1415" upper="3.1415" effort="0" velocity="2.7925"/>
+      <limit lower="-1.5707" upper="1.5707" effort="0" velocity="2.7925"/>
     </joint>
     <joint name="${prefix}joint_4" type="revolute">
@@ -143,5 +143,5 @@
       <origin xyz="0.46 0 0.26" rpy="0 0 0"/>
       <axis xyz="1 0 0"/>
-      <limit lower="-6.2831" upper="6.2831" effort="0" velocity="4.0142"/>
+      <limit lower="-1.5707" upper="1.5707" effort="0" velocity="4.0142"/>
     </joint>
     <joint name="${prefix}joint_5" type="revolute">
@@ -150,5 +150,5 @@
       <origin xyz="0.5 0 0" rpy="0 0 0"/>
       <axis xyz="0 1 0"/>
-      <limit lower="-2.1816" upper="2.1816" effort="0" velocity="4.0142"/>
+      <limit lower="-1.5707" upper="1.5707" effort="0" velocity="4.0142"/>
     </joint>
     <joint name="${prefix}joint_6" type="revolute">
@@ -157,5 +157,5 @@
       <origin xyz="0.7 0 0.01" rpy="0 0 0"/>
       <axis xyz="1 0 0"/>
-      <limit lower="-6.2831" upper="6.2831" effort="0" velocity="6.1086"/>
+      <limit lower="-1.5707" upper="1.5707" effort="0" velocity="6.1086"/>
     </joint>
     <!-- end of joint list -->
